File: tsuka60.kicad_pcb (KiCad board)
At the start: 2 copper layers, 285 x 95.1 mm, 188 parts, among them SW1 SW_Push, U1 ATmega32U4-AU, Y1 Resonator_Small

Commit message: 2/19
Parts:
- added H1: Half Side Hole, acheron_MountingHoles:halfSideHole, F.Cu at (94.8, 169.1)
- added H10: Oval Mounting Hole, acheron_MountingHoles:MoutingHole_Oval_7mm_5.0x2.5mm, F.Cu at (170.7, 121.8)
- added H2: Mounting Hole, acheron_MountingHoles:MoutingHole_Oval_7mm_5.0x2.5mm, F.Cu at (120.0, 140.5)
- added H3: Oval Mounting Hole, acheron_MountingHoles:MoutingHole_Oval_7mm_5.0x2.5mm, F.Cu at (222.8, 159.6)
- added H4: Oval Mounting Hole, acheron_MountingHoles:MoutingHole_Oval_7mm_5.0x2.5mm, F.Cu at (285.3, 197.7)
- added H5: Oval Mounting Hole, acheron_MountingHoles:MoutingHole_Oval_7mm_5.0x2.5mm, F.Cu at (354.8, 140.6)
- added H6: Half Side Hole, acheron_MountingHoles:halfSideHole, F.Cu at (379.8, 169.1)
- added H7: Oval Mounting Hole, acheron_MountingHoles:MoutingHole_Oval_7mm_5.0x2.5mm, F.Cu at (129.0, 194.4)
- added H8: Oval Mounting Hole, acheron_MountingHoles:MoutingHole_Oval_7mm_5.0x2.5mm, F.Cu at (304.0, 121.8)
- added H9: Oval Mounting Hole, acheron_MountingHoles:MoutingHole_Oval_7mm_5.0x2.5mm, F.Cu at (351.6, 193.2)
- added J1: TYPE-C-31-M12_13, acheron_Connectors:TYPE-C-31-M-12, F.Cu at (113.0, 118.3)
- added LED29: YS-SK6812MINI-E, LED_kicad_footprints-master:YS-SK6812MINI-E, B.Cu at (448.6, 20.6)
- MX61-3: footprint MX_Alps_Hybrid:MX-1U-NoLED -> MX_Only:MXOnly-1U-NoLED
- MX75-3: footprint MX_Alps_Hybrid:MX-1U-NoLED -> MX_Only:MXOnly-1U

Commit message: 3/1/2021
Parts:
- removed MX61-1: L-CTRL, MX_Alps_Hybrid:MX-1.25U-NoLED
- removed MX61-3: FN, MX_Only:MXOnly-1U-NoLED
- removed MX62-1: L-WIN, MX_Alps_Hybrid:MX-1.25U-NoLED
- removed MX62-3: CONTROL, MX_Alps_Hybrid:MX-1U-NoLED
- removed MX63-1: L-ALT, MX_Alps_Hybrid:MX-1.25U-NoLED
- removed MX63-3: OPTION, MX_Alps_Hybrid:MX-1U-NoLED
- removed MX64-3, MX65-4, MX71-4: CMD, MX_Alps_Hybrid:MX-1U-NoLED
- removed MX65-1: LEFT SPACE, MX_Alps_Hybrid:MX-2.75U-ReversedStabilizers-NoLED
- removed MX65-2: LEFT SPACE, MX_Alps_Hybrid:MX-3U-ReversedStabilizers-NoLED
- removed MX65-3: LEFT SPACE, MX_Alps_Hybrid:MX-2.75U-NoLED
- removed MX65-5, MX71-5: CMD, MX_Alps_Hybrid:MX-1.25U-NoLED
- removed MX66-4: LEFT SPACE, MX_Alps_Hybrid:MX-2U-ReversedStabilizers-NoLED
- removed MX66-5: LEFT SPACE, MX_Alps_Hybrid:MX-1.25U-NoLED
- removed MX67-5: LEFT CENTRE, MX_Alps_Hybrid:MX-1U-NoLED
- removed MX68: SPACE, MX_Alps_Hybrid:MX-7U-ReversedStabilizers-NoLED
- removed MX68-1: RETURN, MX_Alps_Hybrid:MX-2U-ReversedStabilizers-NoLED
- removed MX69-5: RIGHT CENTRE, MX_Alps_Hybrid:MX-1U-NoLED
- removed MX70-4: RIGHT SPACE, MX_Alps_Hybrid:MX-2U-ReversedStabilizers-NoLED
- removed MX70-5: RIGHT SPACE, MX_Alps_Hybrid:MX-1.25U-NoLED
- removed MX71-1: RIGHT SPACE, MX_Alps_Hybrid:MX-2.75U-ReversedStabilizers-NoLED
- removed MX71-2: RIGHT SPACE, MX_Alps_Hybrid:MX-3U-ReversedStabilizers-NoLED
- removed MX71-3: RIGHT SPACE, MX_Alps_Hybrid:MX-2.75U-NoLED
- removed MX72-3: LEFT, MX_Alps_Hybrid:MX-1U-NoLED
- removed MX73-1: R-ALT, MX_Alps_Hybrid:MX-1.25U-NoLED
- removed MX73-3: DOWN, MX_Alps_Hybrid:MX-1U-NoLED
- removed MX74-1: R-WIN, MX_Alps_Hybrid:MX-1.25U-NoLED
- removed MX74-3: UP, MX_Alps_Hybrid:MX-1U-NoLED
- removed MX75-1: R-CTRL, MX_Alps_Hybrid:MX-1.25U-NoLED
- removed MX75-3: RIGHT, MX_Only:MXOnly-1U
- added ?: , , F.Cu at (-54.0, 97.1)
- added ?: , , F.Cu at (-79.5, 227.4)
- added C10: 0.1uF, Capacitor_SMD:C_0805_2012Metric, F.Cu at (290.3, 70.5)
- added C11: 0.1uF, Capacitor_SMD:C_0805_2012Metric, B.Cu at (199.2, 113.3)
- added C12: 0.1uF, Capacitor_SMD:C_0805_2012Metric, B.Cu at (199.2, 132.4)
- added C13: 0.1uF, Capacitor_SMD:C_0805_2012Metric, B.Cu at (194.5, 151.4)
- added C14: 0.1uF, Capacitor_SMD:C_0805_2012Metric, B.Cu at (208.7, 170.5)
- added C15: 0.1uF, Capacitor_SMD:C_0805_2012Metric, B.Cu at (237.3, 113.4)
- added C16: 0.1uF, Capacitor_SMD:C_0805_2012Metric, B.Cu at (237.3, 132.4)
- added C17: 0.1uF, Capacitor_SMD:C_0805_2012Metric, B.Cu at (237.3, 151.3)
- added C18: 0.1uF, Capacitor_SMD:C_0805_2012Metric, B.Cu at (245.2, 172.2)
- added C19: 0.1uF, Capacitor_SMD:C_0805_2012Metric, B.Cu at (275.4, 113.4)
- added C20: 0.1uF, Capacitor_SMD:C_0805_2012Metric, B.Cu at (275.4, 132.4)
- added C21: 0.1uF, Capacitor_SMD:C_0805_2012Metric, B.Cu at (280.2, 151.4)
- added C22: 0.1uF, Capacitor_SMD:C_0805_2012Metric, B.Cu at (285.6, 189.6)
- added C23: 0.1uF, Capacitor_SMD:C_0805_2012Metric, B.Cu at (285.0, 170.5)
- added C23: 0.1uF, Capacitor_SMD:C_0805_2012Metric, F.Cu at (261.5, 92.3)
- added C24: 0.1uF, Capacitor_SMD:C_0805_2012Metric, B.Cu at (248.5, 191.1)
- added C24: 0.1uF, Capacitor_SMD:C_0805_2012Metric, F.Cu at (266.3, 87.3)
- added C25: 0.1uF, Capacitor_SMD:C_0805_2012Metric, B.Cu at (210.2, 191.1)
- added C25: 0.1uF, Capacitor_SMD:C_0805_2012Metric, F.Cu at (289.2, 64.5)
- added C26: 0.1uF, Capacitor_SMD:C_0805_2012Metric, F.Cu at (266.3, 84.3)
- added C27: 0.1uF, Capacitor_SMD:C_0805_2012Metric, B.Cu at (313.5, 113.4)
- added C28: 0.1uF, Capacitor_SMD:C_0805_2012Metric, B.Cu at (313.5, 132.4)
- added C29: 0.1uF, Capacitor_SMD:C_0805_2012Metric, B.Cu at (318.3, 151.4)
- added C30: 0.1uF, Capacitor_SMD:C_0805_2012Metric, B.Cu at (323.1, 170.5)
- added C31: 0.1uF, Capacitor_SMD:C_0805_2012Metric, B.Cu at (323.1, 189.5)
- added C32: 0.1uF, Capacitor_SMD:C_0805_2012Metric, B.Cu at (361.2, 113.4)
- added C33: 0.1uF, Capacitor_SMD:C_0805_2012Metric, B.Cu at (370.7, 132.4)
- added C34: 0.1uF, Capacitor_SMD:C_0805_2012Metric, B.Cu at (358.8, 151.4)
- added C35: 0.1uF, Capacitor_SMD:C_0805_2012Metric, B.Cu at (365.9, 170.5)
- added C36: 0.1uF, Capacitor_SMD:C_0805_2012Metric, B.Cu at (365.9, 189.5)
- added C6: 0.1uF, Capacitor_SMD:C_0805_2012Metric, F.Cu at (257.0, 90.9)
- added C7: 0.1uF, Capacitor_SMD:C_0805_2012Metric, F.Cu at (283.9, 61.5)
- added C8: 0.1uF, Capacitor_SMD:C_0805_2012Metric, F.Cu at (284.1, 78.4)
- added C9: 0.1uF, Capacitor_SMD:C_0805_2012Metric, F.Cu at (288.4, 61.5)
- added D37: D_Small, Diode_SMD:D_0805_2012Metric, F.Cu at (123.0, -0.79)
- added F2: 500mA, Fuse:Fuse_1206_3216Metric, F.Cu at (265.8, 78.1)
- added J1: USB2_C_Receptacle, Type-C:HRO-TYPE-C-31-M-12-Assembly, F.Cu at (195.3, 64.7)
- added J2: Conn_01x04, random-keyboard-parts:JST-SR-4, F.Cu at (177.2, 63.1)
- added LED1: YS-SK6812MINI-E, LED_kicad_footprints:YS-SK6812MINI-E, F.Cu at (234.5, 88.4)
- added LED10: YS-SK6812MINI-E, LED_kicad_footprints:YS-SK6812MINI-E, B.Cu at (275.4, 115.9)
- added LED11: YS-SK6812MINI-E, LED_kicad_footprints:YS-SK6812MINI-E, B.Cu at (294.5, 115.9)
- added LED12: YS-SK6812MINI-E, LED_kicad_footprints:YS-SK6812MINI-E, B.Cu at (313.5, 115.9)
- added LED13: YS-SK6812MINI-E, LED_kicad_footprints:YS-SK6812MINI-E, B.Cu at (332.6, 115.9)
- added LED19: YS-SK6812MINI-E, LED_kicad_footprints:YS-SK6812MINI-E, B.Cu at (161.1, 134.9)
- added LED2: YS-SK6812MINI-E, LED_kicad_footprints:YS-SK6812MINI-E, F.Cu at (234.5, 80.1)
- added LED20: YS-SK6812MINI-E, LED_kicad_footprints:YS-SK6812MINI-E, B.Cu at (180.2, 134.9)
- added LED21: YS-SK6812MINI-E, LED_kicad_footprints:YS-SK6812MINI-E, B.Cu at (199.2, 134.9)
- added LED22: YS-SK6812MINI-E, LED_kicad_footprints:YS-SK6812MINI-E, B.Cu at (218.3, 134.9)
- added LED23: YS-SK6812MINI-E, LED_kicad_footprints:YS-SK6812MINI-E, B.Cu at (237.3, 134.9)
- added LED24: YS-SK6812MINI-E, LED_kicad_footprints:YS-SK6812MINI-E, B.Cu at (256.4, 134.9)
- added LED25: YS-SK6812MINI-E, LED_kicad_footprints:YS-SK6812MINI-E, B.Cu at (275.4, 134.9)
- added LED26: YS-SK6812MINI-E, LED_kicad_footprints:YS-SK6812MINI-E, B.Cu at (294.5, 134.9)
- added LED27: YS-SK6812MINI-E, LED_kicad_footprints:YS-SK6812MINI-E, B.Cu at (313.5, 134.9)
- added LED28: YS-SK6812MINI-E, LED_kicad_footprints:YS-SK6812MINI-E, B.Cu at (332.6, 134.9)
- added LED3: YS-SK6812MINI-E, LED_kicad_footprints:YS-SK6812MINI-E, F.Cu at (226.4, 88.4)
- added LED30: YS-SK6812MINI-E, LED_kicad_footprints:YS-SK6812MINI-E, B.Cu at (370.7, 134.9)
- added LED33: YS-SK6812MINI-E, LED_kicad_footprints:YS-SK6812MINI-E, F.Cu at (242.6, 74.4)
- added LED34: YS-SK6812MINI-E, LED_kicad_footprints:YS-SK6812MINI-E, B.Cu at (175.4, 154.0)
- added LED35: YS-SK6812MINI-E, LED_kicad_footprints:YS-SK6812MINI-E, B.Cu at (194.5, 154.0)
- added LED36: YS-SK6812MINI-E, LED_kicad_footprints:YS-SK6812MINI-E, B.Cu at (213.5, 154.0)
- added LED38: YS-SK6812MINI-E, LED_kicad_footprints:YS-SK6812MINI-E, B.Cu at (237.3, 154.0)
- added LED39: YS-SK6812MINI-E, LED_kicad_footprints:YS-SK6812MINI-E, B.Cu at (261.1, 154.0)
- added LED4: YS-SK6812MINI-E, LED_kicad_footprints:YS-SK6812MINI-E, B.Cu at (161.1, 115.9)
- added LED40: YS-SK6812MINI-E, LED_kicad_footprints:YS-SK6812MINI-E, B.Cu at (280.2, 154.0)
- added LED404: YS-SK6812MINI-E, LED_kicad_footprints:YS-SK6812MINI-E, F.Cu at (253.3, 62.0)
- added LED41: YS-SK6812MINI-E, LED_kicad_footprints:YS-SK6812MINI-E, B.Cu at (299.2, 154.0)
- added LED42: YS-SK6812MINI-E, LED_kicad_footprints:YS-SK6812MINI-E, B.Cu at (318.3, 154.0)
- added LED43: YS-SK6812MINI-E, LED_kicad_footprints:YS-SK6812MINI-E, B.Cu at (337.3, 154.0)
- added LED44: YS-SK6812MINI-E, LED_kicad_footprints:YS-SK6812MINI-E, B.Cu at (358.8, 154.0)
- added LED45: YS-SK6812MINI-E, LED_kicad_footprints:YS-SK6812MINI-E, B.Cu at (361.2, 115.9)
- added LED49: YS-SK6812MINI-E, LED_kicad_footprints:YS-SK6812MINI-E, B.Cu at (170.7, 173.0)
- added LED5: YS-SK6812MINI-E, LED_kicad_footprints:YS-SK6812MINI-E, B.Cu at (180.2, 115.9)
- added LED50: YS-SK6812MINI-E, LED_kicad_footprints:YS-SK6812MINI-E, B.Cu at (189.7, 173.0)
- added LED505: YS-SK6812MINI-E, LED_kicad_footprints:YS-SK6812MINI-E, F.Cu at (261.4, 57.9)
- added LED51: YS-SK6812MINI-E, LED_kicad_footprints:YS-SK6812MINI-E, B.Cu at (208.8, 173.0)
- added LED52: YS-SK6812MINI-E, LED_kicad_footprints:YS-SK6812MINI-E, B.Cu at (227.8, 174.6)
- added LED54: YS-SK6812MINI-E, LED_kicad_footprints:YS-SK6812MINI-E, B.Cu at (246.9, 174.6)
- added LED55: WS2812B-Worldsemi-unnamed-rescue, LED_kicad_footprints:YS-SK6812MINI-E, B.Cu at (266.0, 173.0)
- added LED56: YS-SK6812MINI-E, LED_kicad_footprints:YS-SK6812MINI-E, B.Cu at (285.0, 173.0)
- added LED57: YS-SK6812MINI-E, LED_kicad_footprints:YS-SK6812MINI-E, B.Cu at (304.0, 173.0)
- added LED58: YS-SK6812MINI-E, LED_kicad_footprints:YS-SK6812MINI-E, B.Cu at (323.1, 173.0)
- added LED59: YS-SK6812MINI-E, LED_kicad_footprints:YS-SK6812MINI-E, B.Cu at (342.1, 173.0)
- added LED6: YS-SK6812MINI-E, LED_kicad_footprints:YS-SK6812MINI-E, B.Cu at (199.2, 115.9)
- added LED60: YS-SK6812MINI-E, LED_kicad_footprints:YS-SK6812MINI-E, B.Cu at (365.9, 173.0)
- added LED64: YS-SK6812MINI-E, LED_kicad_footprints:YS-SK6812MINI-E, F.Cu at (258.9, 66.2)
- added LED65: YS-SK6812MINI-E, LED_kicad_footprints:YS-SK6812MINI-E, B.Cu at (189.7, 192.1)
- added LED66: YS-SK6812MINI-E, LED_kicad_footprints:YS-SK6812MINI-E, B.Cu at (208.8, 193.7)
- added LED67: YS-SK6812MINI-E, LED_kicad_footprints:YS-SK6812MINI-E, B.Cu at (228.4, 193.2)
- added LED69: YS-SK6812MINI-E, LED_kicad_footprints:YS-SK6812MINI-E, B.Cu at (246.9, 193.7)
- added LED7: YS-SK6812MINI-E, LED_kicad_footprints:YS-SK6812MINI-E, B.Cu at (218.3, 115.9)
- added LED70: WS2812B-Worldsemi-unnamed-rescue, LED_kicad_footprints:YS-SK6812MINI-E, B.Cu at (265.9, 193.7)
- added LED71: YS-SK6812MINI-E, LED_kicad_footprints:YS-SK6812MINI-E, B.Cu at (285.6, 192.1)
- added LED72: YS-SK6812MINI-E, LED_kicad_footprints:YS-SK6812MINI-E, B.Cu at (304.0, 192.1)
- added LED73: YS-SK6812MINI-E, LED_kicad_footprints:YS-SK6812MINI-E, B.Cu at (323.1, 192.1)
- added LED74: YS-SK6812MINI-E, LED_kicad_footprints:YS-SK6812MINI-E, B.Cu at (342.1, 192.1)
- added LED75: YS-SK6812MINI-E, LED_kicad_footprints:YS-SK6812MINI-E, B.Cu at (365.9, 192.1)
- added LED8: YS-SK6812MINI-E, LED_kicad_footprints:YS-SK6812MINI-E, B.Cu at (237.3, 115.9)
- added LED9: YS-SK6812MINI-E, LED_kicad_footprints:YS-SK6812MINI-E, B.Cu at (256.4, 115.9)
- added MX64: C, MX_Alps_Hybrid:MX-1U-NoLED, F.Cu at (170.7, 197.6)
- added MX65: LEFT SPACE, MX_Alps_Hybrid:MX-1U-NoLED, F.Cu at (189.7, 197.6)
- added MX66: LEFT SPACE, MX_Alps_Hybrid:MX-1U-NoLED, F.Cu at (208.8, 197.6)
- added MX66-1: LEFT SPACE, MX_Alps_Hybrid:MX-2U-NoLED, F.Cu at (218.3, 197.6)
- added MX67: LEFT CENTRE, MX_Alps_Hybrid:MX-1U-NoLED, F.Cu at (227.8, 197.6)
- added MX69: RIGHT CENTRE, MX_Alps_Hybrid:MX-1U-NoLED, F.Cu at (246.9, 197.6)
- added MX69-1: RIGHT CENTRE, MX_Alps_Hybrid:MX-2U-NoLED, F.Cu at (256.4, 197.6)
- added MX70: RIGHT SPACE, MX_Alps_Hybrid:MX-1U-NoLED, F.Cu at (265.9, 197.6)
- added MX71: RIGHT SPACE, MX_Alps_Hybrid:MX-1U-NoLED, F.Cu at (285.0, 197.6)
- added MX72: LEFT, MX_Alps_Hybrid:MX-1U-NoLED, F.Cu at (304.0, 197.6)
- added R5: 5.1kΩ, Resistor_SMD:R_0805_2012Metric, F.Cu at (275.2, 87.0)
- added R6: 5.1kΩ, Resistor_SMD:R_0805_2012Metric, F.Cu at (279.7, 81.4)
- added R7: 510, Resistor_SMD:R_0805_2012Metric, F.Cu at (288.6, 75.4)
- added U2: SRV05-4, Package_TO_SOT_SMD:SOT-23-6, F.Cu at (257.2, 87.1)
- added U3: ATmega32U4-MU, Package_DFN_QFN:QFN-44-1EP_7x7mm_P0.5mm_EP5.2x5.2mm, B.Cu at (82.2, 179.4)
- LED29: footprint LED_kicad_footprints-master:YS-SK6812MINI-E -> LED_kicad_footprints:YS-SK6812MINI-E
- MX45: footprint MX_Alps_Hybrid:MX-2U-NoLED -> MX_Alps_Hybrid:MX-2U-ReversedStabilizers-NoLED
- MX53: footprint MX_Alps_Hybrid:MX-2U-ReversedStabilizers-NoLED -> MX_Alps_Hybrid:MX-2U-NoLED
- MX63, MX73: footprint MX_Alps_Hybrid:MX-1.5U-NoLED -> MX_Alps_Hybrid:MX-1U-NoLED
- moved LED29 149.9 mm to (351.6, 134.9)
- moved D30 12.0 mm to (364.3, 146.8)
- moved MX63 4.76 mm to (151.6, 197.6), turned to 180 degrees
- moved MX73 4.76 mm to (323.1, 197.6), turned to 180 degrees
- turned MX1 to 180 degrees
- turned MX10 to 180 degrees
- turned MX11 to 180 degrees
- turned MX12 to 180 degrees
- turned MX13 to 180 degrees
- turned MX14 to 180 degrees
- turned MX15 to 180 degrees
- turned MX16 to 180 degrees
- turned MX17 to 180 degrees
- turned MX18 to 180 degrees
- turned MX19 to 180 degrees
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Connections:
- net VCC renamed VBUS
- LED29 pad 1: (no net) -> +5V
- LED29 pad 2: (no net) -> Net-(LED28-Pad4)
- LED29 pad 3: (no net) -> GND
- LED29 pad 4: (no net) -> Net-(LED29-Pad4)
- U1 pad 11: Net-(U1-Pad11) -> LED
Routing:
- net (no net): track 0.00 -> 234.6 mm, vias 0 -> 1
- net Col1: track 149.9 -> 38.8 mm
- net Col2: track 183.3 -> 88.6 mm
- net Col3: track 200.2 -> 110.2 mm
- net Net-(D3-Pad2): track 9.73 -> 93.9 mm
- net Col5: track 265.9 -> 199.7 mm
- net Col4: track 228.7 -> 167.9 mm
- net Net-(D45-Pad2): track 52.4 -> 0.00 mm, vias 1 -> 0
- net Col12: track 332.1 -> 287.5 mm
- net Net-(D36-Pad2): track 9.73 -> 53.7 mm
- net Net-(D35-Pad2): track 9.73 -> 53.7 mm
- net Net-(D58-Pad2): track 9.73 -> 53.6 mm
- net Row0: track 322.4 -> 285.1 mm
- net Col7: track 215.1 -> 177.9 mm
- net Net-(D38-Pad2): track 12.1 -> 49.3 mm
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
Commit message: 3/5/2021
Parts:
- removed ? (x2): , 
- removed the C23 at (261.5, 92.3)
- removed the C24 at (266.3, 87.3)
- removed the C25 at (289.2, 64.5)
- removed the D64 at (153.2, 202.6)
- removed D68: D_Small, Diode_SMD:D_0805_2012Metric
- removed F1: Polyfuse_Small, Fuse:Fuse_1206_3216Metric
- removed the H6 at (379.8, 169.1)
- removed J1: TYPE-C-31-M12_13, acheron_Connectors:TYPE-C-31-M-12
- removed J1: USB2_C_Receptacle, Type-C:HRO-TYPE-C-31-M-12-Assembly
- removed REF**: 60_Outline, Custom:60_Outline-Modded-Extreme-Katana60
- removed U1: ATmega32U4-AU, Package_QFP:TQFP-44_10x10mm_P0.8mm
- added C37: 0.1uF, Capacitor_SMD:C_0805_2012Metric, B.Cu at (123.0, 132.4)
- added C38: 0.1uF, Capacitor_SMD:C_0805_2012Metric, B.Cu at (132.6, 170.5)
- added C39: 0.1uF, Capacitor_SMD:C_0805_2012Metric, B.Cu at (132.5, 189.5)
- added H10: Hole, 2moons:halfSideHole, F.Cu at (379.8, 169.1)
- added LED1: YS-SK6812MINI-E, LED_kicad_footprints:YS-SK6812MINI-E, B.Cu at (104.0, 115.9)
- added LED16: YS-SK6812MINI-E, LED_kicad_footprints:YS-SK6812MINI-E, B.Cu at (104.0, 134.9)
- added LED17: YS-SK6812MINI-E, LED_kicad_footprints:YS-SK6812MINI-E, B.Cu at (123.0, 134.9)
- added LED2: YS-SK6812MINI-E, LED_kicad_footprints:YS-SK6812MINI-E, B.Cu at (123.0, 115.9)
- added LED31: YS-SK6812MINI-E, LED_kicad_footprints:YS-SK6812MINI-E, B.Cu at (111.1, 154.0)
- added LED46: YS-SK6812MINI-E, LED_kicad_footprints:YS-SK6812MINI-E, B.Cu at (108.7, 173.0)
- added LED47: YS-SK6812MINI-E, LED_kicad_footprints:YS-SK6812MINI-E, B.Cu at (132.7, 173.0)
- added LED61: YS-SK6812MINI-E, LED_kicad_footprints:YS-SK6812MINI-E, B.Cu at (108.7, 192.1)
- added LED62: YS-SK6812MINI-E, LED_kicad_footprints:YS-SK6812MINI-E, B.Cu at (132.6, 192.1)
- C10, C26, C6, C7, C8, C9, LED33, LED64, R7: moved to B.Cu
- D64: renamed from D37; moved to B.Cu
- H1: value Half Side Hole -> Hole; footprint acheron_MountingHoles:halfSideHole -> 2moons:halfSideHole
- H2: value Mounting Hole -> Hole; footprint acheron_MountingHoles:MoutingHole_Oval_7mm_5.0x2.5mm -> 2moons:MoutingHole_Oval_7mm_5.0x2.5mm
- H3: renamed from H7; value Oval Mounting Hole -> Hole; footprint acheron_MountingHoles:MoutingHole_Oval_7mm_5.0x2.5mm -> 2moons:2MoutingHole_Oval_7mm_5.0x2.5mm
- H4: renamed from H10; value Oval Mounting Hole -> Hole; footprint acheron_MountingHoles:MoutingHole_Oval_7mm_5.0x2.5mm -> 2moons:MoutingHole_Oval_7mm_5.0x2.5mm
- H5: renamed from H3; value Oval Mounting Hole -> Hole; footprint acheron_MountingHoles:MoutingHole_Oval_7mm_5.0x2.5mm -> 2moons:MoutingHole_Oval_7mm_5.0x2.5mm
- H6: renamed from H4; value Oval Mounting Hole -> Hole; footprint acheron_MountingHoles:MoutingHole_Oval_7mm_5.0x2.5mm -> 2moons:MoutingHole_Oval_7mm_5.0x2.5mm
- H7: renamed from H9; value Oval Mounting Hole -> Hole; footprint acheron_MountingHoles:MoutingHole_Oval_7mm_5.0x2.5mm -> 2moons:3MoutingHole_Oval_7mm_5.0x2.5mm
- H8: value Oval Mounting Hole -> Hole; footprint acheron_MountingHoles:MoutingHole_Oval_7mm_5.0x2.5mm -> 2moons:MoutingHole_Oval_7mm_5.0x2.5mm
- H9: renamed from H5; value Oval Mounting Hole -> Hole; footprint acheron_MountingHoles:MoutingHole_Oval_7mm_5.0x2.5mm -> 2moons:MoutingHole_Oval_7mm_5.0x2.5mm
- LED18: renamed from LED2; moved to B.Cu
- LED3: renamed from LED1; moved to B.Cu
- LED32: renamed from LED3; moved to B.Cu
- LED48: renamed from LED404; moved to B.Cu
- LED63: renamed from LED505; moved to B.Cu
- USB1: value Molex-0548190589 -> HRO-TYPE-C-31-M-12; footprint random-keyboard-parts:Molex-0548190519 -> Type-C:HRO-TYPE-C-31-M-12-HandSoldering
- moved D64 193.3 mm to (160.3, 188.9), turned to 270 degrees
- moved LED63 173.4 mm to (151.6, 192.1)
- moved C10 168.8 mm to (170.6, 189.5)
- moved C9 160.5 mm to (170.6, 170.5)
- moved R6 154.2 mm to (125.9, 93.3)
- moved LED64 153.8 mm to (170.7, 192.1), turned to 180 degrees
- moved LED48 150.5 mm to (151.6, 173.0)
- moved C8 147.2 mm to (156.4, 151.4)
- moved C26 146.3 mm to (123.0, 113.4)
- moved R5 142.5 mm to (133.7, 103.9)
- moved C7 141.8 mm to (161.1, 132.4)
- moved F2 140.9 mm to (126.1, 97.2)
- moved U2 131.4 mm to (126.9, 103.9)
- moved LED33 117.4 mm to (156.4, 154.0), turned to 180 degrees
- moved LED32 110.6 mm to (137.3, 154.0)
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Connections:
- C26 pad 1: GND -> +5V
- LED18 pad 3: Net-(LED2-Pad3) -> GND
- LED30 pad 3: Net-(LED30-Pad3) -> GND
- LED32 pad 3: Net-(LED3-Pad3) -> GND
- LED48 pad 3: Net-(LED404-Pad3) -> GND
- LED74 pad 2: Net-(LED74-Pad2) -> Net-(LED59-Pad4)
- R5 pad 2: Net-(J1-PadA5) -> Net-(R5-Pad2)
- R6 pad 2: Net-(J1-PadB5) -> Net-(R6-Pad2)
- U3 pad 1: Net-(U3-Pad1) -> Row0
- U3 pad 10: Net-(U3-Pad10) -> Col1
- U3 pad 11: Net-(U3-Pad11) -> LED
- U3 pad 13: Net-(U3-Pad13) -> Net-(R1-Pad1)
- U3 pad 14: Net-(U3-Pad14) -> +5V
- U3 pad 15: Net-(U3-Pad15) -> GND
- U3 pad 18: Net-(U3-Pad18) -> Col14
- U3 pad 19: Net-(U3-Pad19) -> Col13
- U3 pad 2: Net-(U3-Pad2) -> +5V
- U3 pad 20: Net-(U3-Pad20) -> Col12
- U3 pad 21: Net-(U3-Pad21) -> Col11
- U3 pad 23: Net-(U3-Pad15) -> GND
- U3 pad 24: Net-(U3-Pad24) -> +5V
- U3 pad 25: Net-(U3-Pad25) -> Col10
- U3 pad 26: Net-(U3-Pad26) -> Col9
- U3 pad 28: Net-(U3-Pad28) -> Col8
- U3 pad 29: Net-(U3-Pad29) -> Col7
- U3 pad 3: Net-(U3-Pad3) -> Net-(R3-Pad1)
- U3 pad 30: Net-(U3-Pad30) -> Col6
- U3 pad 31: Net-(U3-Pad31) -> Col5
- U3 pad 32: Net-(U3-Pad32) -> Col4
- U3 pad 33: Net-(U3-Pad33) -> Net-(R4-Pad2)
- U3 pad 34: Net-(U3-Pad14) -> +5V
- U3 pad 35: Net-(U3-Pad15) -> GND
- U3 pad 37: Net-(U3-Pad37) -> Row3
- U3 pad 38: Net-(U3-Pad38) -> Col3
- U3 pad 39: Net-(U3-Pad39) -> Col2
- U3 pad 4: Net-(U3-Pad4) -> Net-(R2-Pad1)
- U3 pad 40: Net-(U3-Pad40) -> Row4
- U3 pad 41: Net-(U3-Pad41) -> Col0
- U3 pad 43: Net-(U3-Pad15) -> GND
- U3 pad 44: Net-(U3-Pad24) -> +5V
- U3 pad 45: Net-(U3-Pad15) -> GND
- U3 pad 5: Net-(U3-Pad5) -> GND
- U3 pad 6: Net-(U3-Pad6) -> Net-(C1-Pad1)
- U3 pad 7: Net-(U3-Pad7) -> +5V
- U3 pad 8: Net-(U3-Pad8) -> Row1
- U3 pad 9: Net-(U3-Pad9) -> Row2
- USB1 pad 2: Net-(USB1-Pad2) -> VBUS
- USB1 pad 3: D+ -> Net-(USB1-Pad3)
- USB1 pad 4: D- -> Net-(R5-Pad2)
- USB1 pad 5: VBUS -> D-
- USB1 pad 6: Net-(USB1-Pad6) -> D+
- Y1 pad 1: Net-(U1-Pad17) -> Net-(U3-Pad17)
- Y1 pad 3: Net-(U1-Pad16) -> Net-(U3-Pad16)
Routing:
- net +5V: track 146.2 -> 827.6 mm, vias 6 -> 30
- net Col14: track 386.6 -> 92.3 mm
- net Col13: track 354.4 -> 113.4 mm
- net (no net): track 234.6 -> 8.50 mm, vias 1 -> 0
- net Col11: track 299.7 -> 98.6 mm
- net Col10: track 318.9 -> 138.3 mm
- net Col12: track 287.5 -> 107.5 mm
- net Col6: track 212.7 -> 40.8 mm
- net GND: track 79.9 -> 239.1 mm, vias 12 -> 23
- net Col9: track 228.5 -> 77.9 mm
- net Col5: track 199.7 -> 52.8 mm
- net Col7: track 177.9 -> 38.9 mm
- net Col0: track 126.7 -> 0.00 mm, vias 1 -> 0
- net Col4: track 167.9 -> 44.6 mm
- net Col3: track 110.2 -> 2.04 mm
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Other:
- board size 285 x 95.1 mm -> 285 x 94 mm

Commit message: 3/16/2021
Parts:
- added G***: LOGO, graphics:moonlogo, B.Cu at (352.7, 174.5)
- F2, J2, MX46, R5, R6, U2: moved to B.Cu
- moved J2 67.5 mm to (186.2, 130.0), turned to 270 degrees
- moved F2 33.2 mm to (112.8, 127.6)
- moved R6 32.9 mm to (114.3, 124.1), turned to 90 degrees
- moved U2 30.2 mm to (112.9, 130.6)
- moved R5 30.1 mm to (111.5, 124.2), turned to 90 degrees
- moved C4 22.9 mm to (118.7, 174.8)
- moved R1 20.7 mm to (127.9, 163.8), turned to 90 degrees
- moved D44 17.1 mm to (346.1, 151.1), turned to 270 degrees
- moved D42 16.3 mm to (307.9, 151.1), turned to 270 degrees
- moved D41 16.3 mm to (288.9, 151.1), turned to 270 degrees
- moved D39 16.3 mm to (250.9, 151.1), turned to 270 degrees
- moved D40 16.3 mm to (269.9, 151.1), turned to 270 degrees
- moved D43 16.3 mm to (327.1, 151.1), turned to 270 degrees
- moved D34 15.8 mm to (167.2, 151.1), turned to 270 degrees
- moved D36 15.6 mm to (205.3, 151.3), turned to 270 degrees
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Connections:
- LED61 pad 3: Net-(LED61-Pad3) -> GND
Routing:
- net +5V: track 827.6 -> 1740.5 mm, vias 30 -> 71
- net GND: track 239.1 -> 974.8 mm, vias 23 -> 84
- net Col12: track 107.5 -> 425.7 mm, vias 0 -> 1
- net LED: track 0.00 -> 306.1 mm, vias 0 -> 4
- net Col14: track 92.3 -> 357.4 mm, vias 0 -> 1
- net Col13: track 113.4 -> 362.0 mm, vias 1 -> 2
- net Col11: track 98.6 -> 334.1 mm, vias 0 -> 1
- net Col9: track 77.9 -> 300.1 mm, vias 0 -> 1
- net Col7: track 38.9 -> 233.4 mm, vias 0 -> 1
- net Col3: track 2.04 -> 189.8 mm, vias 0 -> 1
- net Col6: track 40.8 -> 226.9 mm, vias 0 -> 1
- net Col10: track 138.3 -> 323.0 mm, vias 0 -> 1
- net Col2: track 0.00 -> 173.8 mm, vias 0 -> 1
- net Col5: track 52.8 -> 224.6 mm, vias 0 -> 1
- net Col8: track 138.1 -> 290.6 mm, vias 0 -> 1
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- added copper zone on B.Cu, net (none)
- added copper zone on F.Cu, net (none)
