File: tsuka60.sch (KiCad schematic (older format))
At the start: 249 parts, among them SW1 SW_Push, U1 ATmega32U4-AU, Y1 Resonator_Small

Commit message: 3/1/2021
Parts:
- removed D64, D68: D_Small, Diode_SMD:D_0805_2012Metric, symbol Device:D_Small
- removed MX61-1: L-CTRL, MX_Alps_Hybrid:MX-1.25U-NoLED, symbol MX_Alps_Hybrid:MX-NoLED
- removed MX61-3: FN, MX_Alps_Hybrid:MX-1U-NoLED, symbol MX_Alps_Hybrid:MX-NoLED
- removed MX62-1: L-WIN, MX_Alps_Hybrid:MX-1.25U-NoLED, symbol MX_Alps_Hybrid:MX-NoLED
- removed MX62-3: CONTROL, MX_Alps_Hybrid:MX-1U-NoLED, symbol MX_Alps_Hybrid:MX-NoLED
- removed MX63-1: L-ALT, MX_Alps_Hybrid:MX-1.25U-NoLED, symbol MX_Alps_Hybrid:MX-NoLED
- removed MX63-3: OPTION, MX_Alps_Hybrid:MX-1U-NoLED, symbol MX_Alps_Hybrid:MX-NoLED
- removed MX64-3, MX65-4, MX71-4: CMD, MX_Alps_Hybrid:MX-1U-NoLED, symbol MX_Alps_Hybrid:MX-NoLED
- removed MX65-2: LEFT SPACE, MX_Alps_Hybrid:MX-3U-ReversedStabilizers-NoLED, symbol MX_Alps_Hybrid:MX-NoLED
- removed MX65-3: LEFT SPACE, MX_Alps_Hybrid:MX-2.75U-NoLED, symbol MX_Alps_Hybrid:MX-NoLED
- removed MX65-5, MX71-5: CMD, MX_Alps_Hybrid:MX-1.25U-NoLED, symbol MX_Alps_Hybrid:MX-NoLED
- removed MX66-5: LEFT SPACE, MX_Alps_Hybrid:MX-1.25U-NoLED, symbol MX_Alps_Hybrid:MX-NoLED
- removed MX68: SPACE, MX_Alps_Hybrid:MX-7U-ReversedStabilizers-NoLED, symbol MX_Alps_Hybrid:MX-NoLED
- removed MX68-1: RETURN, MX_Alps_Hybrid:MX-2U-ReversedStabilizers-NoLED, symbol MX_Alps_Hybrid:MX-NoLED
- removed MX70-5: RIGHT SPACE, MX_Alps_Hybrid:MX-1.25U-NoLED, symbol MX_Alps_Hybrid:MX-NoLED
- removed MX71-2: RIGHT SPACE, MX_Alps_Hybrid:MX-3U-ReversedStabilizers-NoLED, symbol MX_Alps_Hybrid:MX-NoLED
- removed MX71-3: RIGHT SPACE, MX_Alps_Hybrid:MX-2.75U-NoLED, symbol MX_Alps_Hybrid:MX-NoLED
- removed MX73-1: R-ALT, MX_Alps_Hybrid:MX-1.25U-NoLED, symbol MX_Alps_Hybrid:MX-NoLED
- removed MX73-3: DOWN, MX_Alps_Hybrid:MX-1U-NoLED, symbol MX_Alps_Hybrid:MX-NoLED
- removed MX74-1: R-WIN, MX_Alps_Hybrid:MX-1.25U-NoLED, symbol MX_Alps_Hybrid:MX-NoLED
- removed MX74-3: UP, MX_Alps_Hybrid:MX-1U-NoLED, symbol MX_Alps_Hybrid:MX-NoLED
- removed MX75-1: R-CTRL, MX_Alps_Hybrid:MX-1.25U-NoLED, symbol MX_Alps_Hybrid:MX-NoLED
- removed MX75-3: RIGHT, MX_Alps_Hybrid:MX-1U-NoLED, symbol MX_Alps_Hybrid:MX-NoLED
- added C10, C11, C12, C13, C14, C15, C16, C17, C18, C19, C20, C21, C22, C23, C24, C25, C27, C28, C29, C30, C31, C36, C6, C7, C8, C9: 0.1uF, Capacitor_SMD:C_0805_2012Metric, symbol Device:C_Small
- added D37: D_Small, Diode_SMD:D_0805_2012Metric, symbol Device:D_Small
- added LED13, LED28, LED39, LED52, LED56, LED66, LED69, LED72, LED75: YS-SK6812MINI-E, LED_kicad_footprints:YS-SK6812MINI-E, symbol trifecta-rescue:WS2812B-Worldsemi-unnamed-rescue
- added LED70: WS2812B-Worldsemi-unnamed-rescue, LED_kicad_footprints:YS-SK6812MINI-E, symbol trifecta-rescue:WS2812B-Worldsemi-unnamed-rescue
- added MX64: C, MX_Alps_Hybrid:MX-1U-NoLED, symbol MX_Alps_Hybrid:MX-NoLED
- added MX66-1: LEFT SPACE, MX_Alps_Hybrid:MX-2U-NoLED, symbol MX_Alps_Hybrid:MX-NoLED
- added MX69-1: RIGHT CENTRE, MX_Alps_Hybrid:MX-2U-NoLED, symbol MX_Alps_Hybrid:MX-NoLED
- added U3: ATmega32U4-MU, Package_DFN_QFN:QFN-44-1EP_7x7mm_P0.5mm_EP5.2x5.2mm, symbol MCU_Microchip_ATmega:ATmega32U4-MU
- C32, C33, C34, C35: renamed from C?; footprint (none) -> Capacitor_SMD:C_0805_2012Metric
- J1: renamed from J?; footprint (none) -> Type-C:HRO-TYPE-C-31-M-12-Assembly
- J2: renamed from J?; footprint (none) -> random-keyboard-parts:JST-SR-4
- LED10, LED11, LED12, LED18, LED19, LED20, LED21, LED22, LED23, LED24, LED25, LED26, LED27, LED29, LED3, LED30, LED32, LED33, LED34, LED35, LED36, LED38, LED4, LED40, LED41, LED42, LED43, LED44, LED45, LED48, LED49, LED5, LED50, LED51, LED54, LED57, LED58, LED59, LED6, LED60, LED63, LED64, LED65, LED67, LED7, LED71, LED73, LED74, LED8, LED9: renamed from LED?; value WS2812B-Worldsemi-unnamed-rescue -> YS-SK6812MINI-E; footprint LEDs:LED_WS2812B-PLCC4 -> LED_kicad_footprints:YS-SK6812MINI-E
- LED55: renamed from LED?; footprint LEDs:LED_WS2812B-PLCC4 -> LED_kicad_footprints:YS-SK6812MINI-E
- MX45: footprint MX_Alps_Hybrid:MX-2U-NoLED -> MX_Alps_Hybrid:MX-2U-ReversedStabilizers-NoLED
- MX53: footprint MX_Alps_Hybrid:MX-2U-ReversedStabilizers-NoLED -> MX_Alps_Hybrid:MX-2U-NoLED
- MX63, MX73: footprint MX_Alps_Hybrid:MX-1.5U-NoLED -> MX_Alps_Hybrid:MX-1U-NoLED
- MX65: renamed from MX65-1; footprint MX_Alps_Hybrid:MX-2.75U-ReversedStabilizers-NoLED -> MX_Alps_Hybrid:MX-1U-NoLED
- MX66: renamed from MX66-4; footprint MX_Alps_Hybrid:MX-2U-ReversedStabilizers-NoLED -> MX_Alps_Hybrid:MX-1U-NoLED
- MX70: renamed from MX70-4; footprint MX_Alps_Hybrid:MX-2U-ReversedStabilizers-NoLED -> MX_Alps_Hybrid:MX-1U-NoLED
- MX71: renamed from MX71-1; footprint MX_Alps_Hybrid:MX-2.75U-ReversedStabilizers-NoLED -> MX_Alps_Hybrid:MX-1U-NoLED
- R5, R6, R7: renamed from R?; footprint (none) -> Resistor_SMD:R_0805_2012Metric
- gave numbers to parts that had none: 2
- renumbered MX67-5 to MX67, MX69-5 to MX69, MX72-3 to MX72
Connections:
- net +5V: now also J2.1 (Pin_1), LED10.1 (VDD), LED11.1 (VDD), LED12.1 (VDD), LED18.1 (VDD), LED19.1 (VDD), LED20.1 (VDD), LED21.1 (VDD), LED22.1 (VDD), LED23.1 (VDD), LED24.1 (VDD), LED25.1 (VDD), LED26.1 (VDD), LED27.1 (VDD), LED3.1 (VDD), LED32.1 (VDD), LED33.1 (VDD), LED34.1 (VDD), LED35.1 (VDD), LED36.1 (VDD), LED38.1 (VDD), LED4.1 (VDD), LED40.1 (VDD), LED41.1 (VDD), LED42.1 (VDD), LED48.1 (VDD), LED49.1 (VDD), LED5.1 (VDD), LED50.1 (VDD), LED51.1 (VDD), LED54.1 (VDD), LED55.1 (VDD), LED57.1 (VDD), LED58.1 (VDD), LED6.1 (VDD), LED63.1 (VDD), LED64.1 (VDD), LED65.1 (VDD), LED67.1 (VDD), LED7.1 (VDD), LED71.1 (VDD), LED73.1 (VDD), LED8.1 (VDD), LED9.1 (VDD), C10.1, C11.1, C12.1, C13.1, C14.1, C15.1, C16.1, C17.1, C18.1, C19.1, C20.1, C21.1, C22.1, C23.1, C24.1, C25.1, C27.1, C28.1, C29.1, C30.1, C31.1, C36.1, C6.1, C7.1, C8.1, C9.1, LED13.1 (VDD), LED28.1 (VDD), LED39.1 (VDD), LED52.1 (VDD), LED56.1 (VDD), LED66.1 (VDD), LED69.1 (VDD), LED70.1 (VDD), LED72.1 (VDD), LED75.1 (VDD)
- net Col3: now also MX64.1 (COL)
- net Col5: now also MX66-1.1 (COL)
- net Col8: now also MX69-1.1 (COL)
- net D+: now also J2.3 (Pin_3)
- net D-: now also J2.2 (Pin_2)
- net GND: now also J2.4 (Pin_4), LED10.3 (VSS), LED11.3 (VSS), LED12.3 (VSS), LED19.3 (VSS), LED20.3 (VSS), LED21.3 (VSS), LED22.3 (VSS), LED23.3 (VSS), LED24.3 (VSS), LED25.3 (VSS), LED26.3 (VSS), LED27.3 (VSS), LED29.3 (VSS), LED3.3 (VSS), LED33.3 (VSS), LED34.3 (VSS), LED35.3 (VSS), LED36.3 (VSS), LED38.3 (VSS), LED4.3 (VSS), LED40.3 (VSS), LED41.3 (VSS), LED42.3 (VSS), LED43.3 (VSS), LED49.3 (VSS), LED5.3 (VSS), LED50.3 (VSS), LED51.3 (VSS), LED54.3 (VSS), LED55.3 (VSS), LED57.3 (VSS), LED58.3 (VSS), LED59.3 (VSS), LED6.3 (VSS), LED63.3 (VSS), LED64.3 (VSS), LED65.3 (VSS), LED67.3 (VSS), LED7.3 (VSS), LED71.3 (VSS), LED73.3 (VSS), LED74.3 (VSS), LED8.3 (VSS), LED9.3 (VSS), C10.2, C11.2, C12.2, C13.2, C14.2, C15.2, C16.2, C17.2, C18.2, C19.2, C20.2, C21.2, C22.2, C23.2, C24.2, C25.2, C27.2, C28.2, C29.2, C30.2, C31.2, C36.2, C6.2, C7.2, C8.2, C9.2, LED13.3 (VSS), LED28.3 (VSS), LED39.3 (VSS), LED52.3 (VSS), LED56.3 (VSS), LED66.3 (VSS), LED69.3 (VSS), LED70.3 (VSS), LED72.3 (VSS), LED75.3 (VSS)
- net Row4: now also D37.1 (K)
- net at D69.2 (A), MX69.2 (ROW): now also MX69-1.2 (ROW)
- net at D66.2 (A), MX66.2 (ROW): now also MX66-1.2 (ROW)
- net at LED29.2 (DOUT): now also LED28.4 (DIN)
- net at LED59.4 (DIN): no longer LED74.2 (DOUT)
- net at LED12.2 (DOUT): now also LED27.4 (DIN)
- net at LED12.4 (DIN): now also LED13.2 (DOUT)
- net at LED27.2 (DOUT): now also LED42.4 (DIN)
- net at LED42.2 (DOUT): now also LED58.4 (DIN)
- net at LED58.2 (DOUT): now also LED73.4 (DIN)
- net at LED11.2 (DOUT): now also LED10.4 (DIN)
- net at LED11.4 (DIN): now also LED26.2 (DOUT)
- net at LED26.4 (DIN): now also LED41.2 (DOUT)
- net at LED41.4 (DIN): now also LED57.2 (DOUT)
- net at LED57.4 (DIN): now also LED72.2 (DOUT)
- net at LED10.2 (DOUT): now also LED25.4 (DIN)
- net at LED25.2 (DOUT): now also LED40.4 (DIN)
- net at LED40.2 (DOUT): now also LED56.4 (DIN)
- net at LED9.2 (DOUT): now also LED8.4 (DIN)
- net at LED9.4 (DIN): now also LED24.2 (DOUT)
- net at LED24.4 (DIN): now also LED39.2 (DOUT)
- net at LED55.2 (DOUT): now also LED39.4 (DIN)
- net at LED55.4 (DIN): now also LED70.2 (DOUT)
- net at LED8.2 (DOUT): now also LED23.4 (DIN)
- net at LED23.2 (DOUT): now also LED38.4 (DIN)
- net at LED38.2 (DOUT): now also LED54.4 (DIN)
- net at LED54.2 (DOUT): now also LED69.4 (DIN)
- net at LED7.2 (DOUT): now also LED6.4 (DIN)
- net at LED7.4 (DIN): now also LED22.2 (DOUT)
- net at LED22.4 (DIN): now also LED36.2 (DOUT)
- net at LED36.4 (DIN): now also LED52.2 (DOUT)
- net at LED67.2 (DOUT): now also LED52.4 (DIN)
- net at LED67.4 (DIN): now also LED69.2 (DOUT)
- net at LED6.2 (DOUT): now also LED21.4 (DIN)
- net at LED21.2 (DOUT): now also LED35.4 (DIN)
- net at LED35.2 (DOUT): now also LED51.4 (DIN)
- net at LED51.2 (DOUT): now also LED66.4 (DIN)
- net at LED5.2 (DOUT): now also LED4.4 (DIN)
- net at LED5.4 (DIN): now also LED20.2 (DOUT)
- net at LED20.4 (DIN): now also LED34.2 (DOUT)
- net at LED34.4 (DIN): now also LED50.2 (DOUT)
- net at LED50.4 (DIN): now also LED65.2 (DOUT)
- net at LED4.2 (DOUT): now also LED19.4 (DIN)
- net at LED19.2 (DOUT): now also LED33.4 (DIN)
- net at LED33.2 (DOUT): now also LED49.4 (DIN)
- net at LED49.2 (DOUT): now also LED64.4 (DIN)
- net at LED3.4 (DIN): now also LED18.2 (DOUT)
- net at LED18.4 (DIN): now also LED32.2 (DOUT)
- net at LED32.4 (DIN): now also LED48.2 (DOUT)
- net at LED48.4 (DIN): now also LED63.2 (DOUT)
- net at LED60.2 (DOUT): now also LED75.4 (DIN); no longer LED74.4 (DIN)
- net at LED73.2 (DOUT): now also LED72.4 (DIN)
- net at LED71.2 (DOUT): now also LED70.4 (DIN)
- net at LED71.4 (DIN): now also LED56.2 (DOUT)
- net at LED65.4 (DIN): now also LED66.2 (DOUT)
- net at LED64.2 (DOUT): now also LED63.4 (DIN)
- new net: D37.2 (A), MX64.2 (ROW)
- new net: LED74.4 (DIN), LED75.2 (DOUT)
- new net: U3.14 (VCC), U3.34 (VCC)
- new net: U3.15 (GND), U3.23 (GND), U3.35 (GND), U3.43 (GND), U3.45 (GND)
- new net: U3.24 (AVCC), U3.44 (AVCC)
- new net: LED13.4 (DIN), LED28.2 (DOUT)
- no-connect marks 2 -> 3
Other:
- moved on the sheet: J2, LED10, LED18, LED19, LED20, LED21, LED22, LED23, LED24, LED25, LED29, LED3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

Commit message: 3/5/2021
Parts:
- removed F1: Polyfuse_Small, Fuse:Fuse_1206_3216Metric, symbol Device:Polyfuse_Small
- removed J1: USB2_C_Receptacle, Type-C:HRO-TYPE-C-31-M-12-Assembly, symbol usb-type-c:USB2_C_Receptacle
- removed U1: ATmega32U4-AU, Package_QFP:TQFP-44_10x10mm_P0.8mm, symbol tsuka60-rescue:ATmega32U4-AU-MCU_Microchip_ATmega
- removed USB1: Molex-0548190589, random-keyboard-parts:Molex-0548190519, symbol random-keyboard-parts:Molex-0548190589
- added C26, C37, C38, C39: 0.1uF, Capacitor_SMD:C_0805_2012Metric, symbol Device:C_Small
- added H1, H10: Hole, 2moons:halfSideHole, symbol keebio:Hole
- added H2, H4, H5, H6, H8, H9: Hole, 2moons:MoutingHole_Oval_7mm_5.0x2.5mm, symbol keebio:Hole
- added H3: Hole, 2moons:2MoutingHole_Oval_7mm_5.0x2.5mm, symbol keebio:Hole
- added H7: Hole, 2moons:3MoutingHole_Oval_7mm_5.0x2.5mm, symbol keebio:Hole
- added LED1, LED16, LED17, LED2, LED31, LED46, LED47, LED61, LED62: YS-SK6812MINI-E, LED_kicad_footprints:YS-SK6812MINI-E, symbol trifecta-rescue:WS2812B-Worldsemi-unnamed-rescue
- added USB1: HRO-TYPE-C-31-M-12, Type-C:HRO-TYPE-C-31-M-12-HandSoldering, symbol keebio:HRO-TYPE-C-31-M-12
- renumbered D37 to D64
Connections:
- net +5V: now also U3.14 (VCC), U3.2 (UVCC), U3.24 (AVCC), U3.34 (VCC), U3.44 (AVCC), U3.7 (VBUS), C26.1, C37.1, C38.1, C39.1, LED1.1 (VDD), LED16.1 (VDD), LED17.1 (VDD), LED2.1 (VDD), LED31.1 (VDD), LED46.1 (VDD), LED47.1 (VDD), LED61.1 (VDD), LED62.1 (VDD)
- net Col0: now also U3.41 (PF0)
- net Col1: now also U3.10 (PB2)
- net Col10: now also U3.25 (PD4)
- net Col11: now also U3.21 (PD3)
- net Col12: now also U3.20 (PD2)
- net Col13: now also U3.19 (PD1)
- net Col14: now also U3.18 (PD0)
- net Col2: now also U3.39 (PF4)
- net Col3: now also U3.38 (PF5)
- net Col4: now also U3.32 (PC7)
- net Col5: now also U3.31 (PC6)
- net Col6: now also U3.30 (PB6)
- net Col7: now also U3.29 (PB5)
- net Col8: now also U3.28 (PB4)
- net Col9: now also U3.26 (PD6)
- net D+: now also USB1.6 (DP1), USB1.8 (DP2)
- net D-: now also USB1.5 (DN2), USB1.7 (DN1)
- net GND: now also LED18.3 (VSS), LED30.3 (VSS), LED32.3 (VSS), LED48.3 (VSS), U3.15 (GND), U3.23 (GND), U3.35 (GND), U3.43 (GND), U3.45 (GND), U3.5 (UGND), C26.2, C37.2, C38.2, C39.2, LED1.3 (VSS), LED16.3 (VSS), LED17.3 (VSS), LED2.3 (VSS), LED31.3 (VSS), LED46.3 (VSS), LED47.3 (VSS), LED62.3 (VSS), USB1.1 (GND), USB1.12 (GND), USB1.13 (SHIELD)
- net LED: now also U3.11 (PB3)
- net Row0: now also U3.1 (PE6)
- net Row1: now also U3.8 (PB0)
- net Row2: now also U3.9 (PB1)
- net Row3: now also U3.37 (PF6)
- net Row4: now also U3.40 (PF1)
- net VCC: now also USB1.11 (VBUS), USB1.2 (VBUS)
- net at R1.1, SW1.2: now also U3.13 (~RESET)
- net at Y1.3: now also U3.16 (XTAL2)
- net at Y1.1: now also U3.17 (XTAL1)
- net at R3.1: now also U3.3 (D-)
- net at R4.2: now also U3.33 (~HWB~/PE2)
- net at R2.1: now also U3.4 (D+)
- net at C1.1: now also U3.6 (UCAP)
- net at LED59.4 (DIN): now also LED74.2 (DOUT)
- net at LED3.2 (DOUT): now also LED2.4 (DIN)
- net at R5.2: now also USB1.4 (CC1)
- net at R6.2: now also USB1.10 (CC2)
- new net: LED17.4 (DIN), LED2.2 (DOUT)
- new net: LED17.2 (DOUT), LED47.4 (DIN)
- new net: LED47.2 (DOUT), LED62.4 (DIN)
- new net: LED61.4 (DIN), LED62.2 (DOUT)
- new net: LED46.4 (DIN), LED61.2 (DOUT)
- new net: LED31.4 (DIN), LED46.2 (DOUT)
- new net: LED16.4 (DIN), LED31.2 (DOUT)
- new net: LED1.4 (DIN), LED16.2 (DOUT)
- no-connect marks 3 -> 4
Other:
- note added: "Mounting Holes"
- moved on the sheet: C1, F2, J2, R1, R2, R3, R4, R5, R6, SW1, U2, U3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

Commit message: 3/16/2021
Connections:
- net GND: now also LED61.3 (VSS)
- no-connect marks 4 -> 8
Changed lines of the file:
@@
 Wire Wire Line
 	12250 10700 12250 11200
-Wire Wire Line
-	12425 12675 12250 12675
 Connection ~ 12250 12675
 Wire Wire Line
@@
 Wire Wire Line
 	26400 12825 26400 13050
+NoConn ~ 6200 13800
+NoConn ~ 6200 14000
+NoConn ~ 6200 15000
+NoConn ~ 6200 12800
+Wire Wire Line
+	12250 12675 12450 12675
 $EndSCHEMATC
